File: board/AugerBoard.kicad_sch (KiCad schematic)
At the start: 0 parts

Commit message: Test commit
Other:
- note added: "Test"
Changed lines of the file:
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@@
 	(generator_version "9.0")
 	(paper "A4")
+	(text "Test"
+		(exclude_from_sim no)
+		(at 79.248 61.722 0)
+		(effects
+			(font
+				(size 1.27 1.27)
+			)
+		)
+	)
 	(sheet_instances
 		(path "/"

Commit message: Main Components
started working on main components
Other:
- added sheet AF interface (AFI.kicad_sch)
- added sheet Communications (communications.kicad_sch)
- added sheet Direction Switch (direction_switch.kicad_sch)
- added sheet Power (power.kicad_sch)
- added sheet Servos (servos.kicad_sch)
- added sheet Soil Sensors (soil_sensors.kicad_sch)
- added sheet Teensy (teensy.kicad_sch)
- added sheet Test Buttons (test_buttons.kicad_sch)
- added sheet VESC (VESC.kicad_sch)
- added sheet mount (mount.kicad_sch)
- note removed: "Test"
