File: board/AugerBoard.kicad_sch (KiCad schematic)
At the start: 0 parts

Commit message: Redesigning Layout
Other:
- sheet Soil Sensors & NPK renamed Soil Sensors
- sheet Power ports: added Spare12VLED, SpareLED1, SpareLED2; removed AFSpareLED, CacheSpareLED, SpareMotorLED
- sheet Servos ports: added SparePWM1, SparePWM2; removed AFSparePWM, SoilCacheSparePWM
- sheet Soil Sensors ports: added none; removed DE, DI, RE, RO
- sheet Teensy ports: added Spare12VLED, SpareLED1, SpareLED2, SparePWM1, SparePWM2, SpareSW1, SpareSW2; removed AFSpareLED, AFSparePWM, AFSpareSW, CacheSpareLED, DE, DI, RE, RO, SCacheSpareSW, SoilCacheSparePWM, SpareMotorLED
- sheet Test Buttons ports: added SpareSW1, SpareSW2; removed AFSpareSW, SCacheSpareSW
Changed lines of the file:
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@@
-	(wire
-		(pts
-			(xy 161.29 93.98) (xy 166.37 93.98)
-		)
-		(stroke
-			(width 0)
-			(type default)
-		)
-	)
 	(wire
 		(pts
@@
 	(wire
 		(pts
-			(xy 161.29 91.44) (xy 166.37 91.44)
-		)
-		(stroke
-			(width 0)
-			(type default)
-		)
-	)
-	(wire
-		(pts
 			(xy 101.6 91.44) (xy 106.68 91.44)
 		)
@@
 		(pts
 			(xy 149.86 125.73) (xy 149.86 130.81)
-		)
-		(stroke
-			(width 0)
-			(type default)
-		)
-	)
-	(wire
-		(pts
-			(xy 161.29 86.36) (xy 166.37 86.36)
-		)
-		(stroke
-			(width 0)
-			(type default)
-		)
-	)
-	(wire
-		(pts
-			(xy 161.29 88.9) (xy 166.37 88.9)
 		)
 		(stroke
@@
 			)
 		)
-		(pin "SoilCacheSparePWM" output
+		(pin "SparePWM1" output
 			(at 106.68 86.36 180)
 			(effects
@@
 			)
 		)
-		(pin "AFSparePWM" output
+		(pin "SparePWM2" output
 			(at 106.68 88.9 180)
 			(effects
@@
 			)
 		)
-		(pin "DE" output
-			(at 161.29 86.36 0)
-			(effects
-				(font
-					(size 1.27 1.27)
-				)
-				(justify right)
-			)
-		)
-		(pin "DI" output
-			(at 161.29 88.9 0)
-			(effects
-				(font
-					(size 1.27 1.27)
-				)
-				(justify right)
-			)
-		)
-		(pin "RE" output
-			(at 161.29 91.44 0)
-			(effects
-				(font
-					(size 1.27 1.27)
-				)
-				(justify right)
-			)
-		)
-		(pin "RO" input
-			(at 161.29 93.98 0)
-			(effects
-				(font
-					(size 1.27 1.27)
-				)
-				(justify right)
-			)
-		)
 		(pin "Moisture" input
 			(at 161.29 99.06 0)
@@
 			)
 		)
-		(pin "SpareMotorLED" output
+		(pin "Spare12VLED" output
 			(at 157.48 125.73 270)
 			(effects
@@
 			)
 		)
-		(pin "AFSpareSW" input
+		(pin "SpareSW1" input
 			(at 106.68 116.84 180)
 			(effects
@@
 			)
 		)
-		(pin "SCacheSpareSW" input
+		(pin "SpareSW2" input
 			(at 106.68 119.38 180)
 			(effects
@@
 			)
 		)
-		(pin "AFSpareLED" output
+		(pin "SpareLED1" output
 			(at 149.86 125.73 270)
 			(effects
@@
 			)
 		)
-		(pin "CacheSpareLED" output
+		(pin "SpareLED2" output
 			(at 147.32 125.73 270)
 			(effects
@@
 			)
 		)
-		(pin "SpareMotorLED" input
+		(pin "Spare12VLED" input
 			(at 157.48 130.81 90)
 			(effects
@@
 			)
 		)
-		(pin "AFSpareLED" input
+		(pin "SpareLED1" input
 			(at 149.86 130.81 90)
 			(effects
@@
 			)
 		)
-		(pin "CacheSpareLED" input
+		(pin "SpareLED2" input
 			(at 147.32 130.81 90)
 			(effects
@@
 			)
 		)
-		(pin "SoilCacheSparePWM" input
+		(pin "SparePWM1" input
 			(at 101.6 86.36 0)
 			(effects
@@
 			)
 		)
-		(pin "AFSparePWM" input
+		(pin "SparePWM2" input
 			(at 101.6 88.9 0)
 			(effects
@@
 			)
 		)
-		(pin "AFSpareSW" output
+		(pin "SpareSW1" output
 			(at 101.6 116.84 0)
 			(effects
@@
 			)
 		)
-		(pin "SCacheSpareSW" output
+		(pin "SpareSW2" output
 			(at 101.6 119.38 0)
 			(effects
@@
 			(color 0 0 0 0.0000)
 		)
-		(property "Sheetname" "Soil Sensors & NPK"
+		(property "Sheetname" "Soil Sensors"
 			(at 166.37 79.2984 0)
 			(effects
@@
 			)
 		)
-		(pin "DE" input
-			(at 166.37 86.36 180)
-			(effects
-				(font
-					(size 1.27 1.27)
-				)
-				(justify left)
-			)
-		)
-		(pin "DI" input
-			(at 166.37 88.9 180)
-			(effects
-				(font
-					(size 1.27 1.27)
-				)
-				(justify left)
-			)
-		)
-		(pin "RE" input
-			(at 166.37 91.44 180)
-			(effects
-				(font
-					(size 1.27 1.27)
-				)
-				(justify left)
-			)
-		)
-		(pin "RO" output
-			(at 166.37 93.98 180)
-			(effects
-				(font
-					(size 1.27 1.27)
-				)
-				(justify left)
-			)
-		)
