File: board/VESC.kicad_sch (KiCad schematic)
At the start: 0 parts

Commit message: Added Parts, Renamed Parts
Added in switches, buttons, & multiple anderson connections for power.
Parts:
- added Conn8: AndersonPP, symbol MRDT_Connectors:AndersonPP
Connections:
- new net +12V: Conn8.2 (V+Log)
- new net GND: Conn8.1 (GND)
