File: board/teensy.kicad_sch (KiCad schematic)
At the start: 1 part, among them U2 Teensy4.1_DEV-16771

Commit message: added pin for AF, added gimbal names, refined look
Connections:
- net AFWhiteLED: now reaches U2.31 (CTX3)
- net ServoSpareLED1 renamed GimbalPanLED
- net ServoSpareLED2 renamed GimbalTiltLED
- net SparePWM1 renamed SciGimbalPan
- net SparePWM2 renamed SciGimbalTilt
- net SpareSW1 renamed GimbalPanSW
- net SpareSW2 renamed GimbalTiltSW
- no-connect marks 10 -> 9
Changed lines of the file:
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@@
-	)
-	(no_connect
-		(at 124.46 91.44)
 	)
 	(no_connect
@@
 	(wire
 		(pts
+			(xy 120.65 99.06) (xy 124.46 99.06)
+		)
+		(stroke
+			(width 0)
+			(type default)
+		)
+	)
+	(wire
+		(pts
+			(xy 165.1 76.2) (xy 168.91 76.2)
+		)
+		(stroke
+			(width 0)
+			(type default)
+		)
+	)
+	(wire
+		(pts
+			(xy 165.1 134.62) (xy 170.18 134.62)
+		)
+		(stroke
+			(width 0)
+			(type default)
+		)
+	)
+	(wire
+		(pts
+			(xy 120.65 88.9) (xy 124.46 88.9)
+		)
+		(stroke
+			(width 0)
+			(type default)
+		)
+	)
+	(wire
+		(pts
+			(xy 165.1 137.16) (xy 170.18 137.16)
+		)
+		(stroke
+			(width 0)
+			(type default)
+		)
+	)
+	(wire
+		(pts
+			(xy 120.65 71.12) (xy 124.46 71.12)
+		)
+		(stroke
+			(width 0)
+			(type default)
+		)
+	)
+	(wire
+		(pts
+			(xy 120.65 83.82) (xy 124.46 83.82)
+		)
+		(stroke
+			(width 0)
+			(type default)
+		)
+	)
+	(wire
+		(pts
+			(xy 165.1 55.88) (xy 168.91 55.88)
+		)
+		(stroke
+			(width 0)
+			(type default)
+		)
+	)
+	(wire
+		(pts
+			(xy 119.38 49.53) (xy 119.38 53.34)
+		)
+		(stroke
+			(width 0)
+			(type default)
+		)
+	)
+	(wire
+		(pts
+			(xy 165.1 116.84) (xy 168.91 116.84)
+		)
+		(stroke
+			(width 0)
+			(type default)
+		)
+	)
+	(wire
+		(pts
+			(xy 165.1 53.34) (xy 168.91 53.34)
+		)
+		(stroke
+			(width 0)
+			(type default)
+		)
+	)
+	(wire
+		(pts
+			(xy 120.65 101.6) (xy 124.46 101.6)
+		)
+		(stroke
+			(width 0)
+			(type default)
+		)
+	)
+	(wire
+		(pts
+			(xy 165.1 114.3) (xy 168.91 114.3)
+		)
+		(stroke
+			(width 0)
+			(type default)
+		)
+	)
+	(wire
+		(pts
+			(xy 165.1 88.9) (xy 168.91 88.9)
+		)
+		(stroke
+			(width 0)
+			(type default)
+		)
+	)
+	(wire
+		(pts
+			(xy 120.65 86.36) (xy 124.46 86.36)
+		)
+		(stroke
+			(width 0)
+			(type default)
+		)
+	)
+	(wire
+		(pts
 			(xy 165.1 78.74) (xy 168.91 78.74)
 		)
@@
 	(wire
 		(pts
-			(xy 120.65 99.06) (xy 124.46 99.06)
-		)
-		(stroke
-			(width 0)
-			(type default)
-		)
-	)
-	(wire
-		(pts
-			(xy 165.1 76.2) (xy 168.91 76.2)
-		)
-		(stroke
-			(width 0)
-			(type default)
-		)
-	)
-	(wire
-		(pts
-			(xy 165.1 134.62) (xy 170.18 134.62)
-		)
-		(stroke
-			(width 0)
-			(type default)
-		)
-	)
-	(wire
-		(pts
-			(xy 120.65 88.9) (xy 124.46 88.9)
-		)
-		(stroke
-			(width 0)
-			(type default)
-		)
-	)
-	(wire
-		(pts
-			(xy 165.1 137.16) (xy 170.18 137.16)
-		)
-		(stroke
-			(width 0)
-			(type default)
-		)
-	)
-	(wire
-		(pts
-			(xy 120.65 71.12) (xy 124.46 71.12)
-		)
-		(stroke
-			(width 0)
-			(type default)
-		)
-	)
-	(wire
-		(pts
-			(xy 120.65 83.82) (xy 124.46 83.82)
-		)
-		(stroke
-			(width 0)
-			(type default)
-		)
-	)
-	(wire
-		(pts
-			(xy 165.1 55.88) (xy 168.91 55.88)
-		)
-		(stroke
-			(width 0)
-			(type default)
-		)
-	)
-	(wire
-		(pts
-			(xy 119.38 49.53) (xy 119.38 53.34)
-		)
-		(stroke
-			(width 0)
-			(type default)
-		)
-	)
-	(wire
-		(pts
-			(xy 165.1 116.84) (xy 168.91 116.84)
-		)
-		(stroke
-			(width 0)
-			(type default)
-		)
-	)
-	(wire
-		(pts
-			(xy 165.1 53.34) (xy 168.91 53.34)
-		)
-		(stroke
-			(width 0)
-			(type default)
-		)
-	)
-	(wire
-		(pts
-			(xy 120.65 101.6) (xy 124.46 101.6)
-		)
-		(stroke
-			(width 0)
-			(type default)
-		)
-	)
-	(wire
-		(pts
-			(xy 165.1 114.3) (xy 168.91 114.3)
-		)
-		(stroke
-			(width 0)
-			(type default)
-		)
-	)
-	(wire
-		(pts
-			(xy 165.1 88.9) (xy 168.91 88.9)
-		)
-		(stroke
-			(width 0)
-			(type default)
-		)
-	)
-	(wire
-		(pts
-			(xy 120.65 86.36) (xy 124.46 86.36)
-		)
-		(stroke
-			(width 0)
-			(type default)
-		)
-	)
-	(wire
-		(pts
 			(xy 120.65 81.28) (xy 124.46 81.28)
 		)
@@
 	(wire
 		(pts
+			(xy 120.65 91.44) (xy 124.46 91.44)
+		)
+		(stroke
+			(width 0)
+			(type default)
+		)
+	)
+	(wire
+		(pts
 			(xy 120.65 116.84) (xy 124.46 116.84)
 		)
@@
 		)
 	)
-	(hierarchical_label "SparePWM2"
+	(hierarchical_label "SciGimbalTilt"
 		(shape output)
 		(at 168.91 78.74 0)
@@
 		)
 	)
+	(hierarchical_label "AFWhiteLED"
+		(shape output)
+		(at 120.65 91.44 180)
+		(effects
+			(font
+				(size 1.27 1.27)
+			)
+			(justify right)
+		)
+	)
 	(hierarchical_label "AFLED340"
 		(shape output)
@@
 		)
 	)
-	(hierarchical_label "SpareSW2"
+	(hierarchical_label "GimbalTiltSW"
 		(shape input)
 		(at 120.65 83.82 180)
@@
 		)
 	)
-	(hierarchical_label "ServoSpareLED1"
+	(hierarchical_label "GimbalPanLED"
 		(shape output)
 		(at 168.91 124.46 0)
@@
 		)
 	)
-	(hierarchical_label "ServoSpareLED2"
+	(hierarchical_label "GimbalTiltLED"
 		(shape output)
 		(at 120.65 73.66 180)
@@
 		)
 	)
-	(hierarchical_label "SparePWM1"
+	(hierarchical_label "SciGimbalPan"
 		(shape output)
 		(at 168.91 127 0)
@@
 		)
 	)
-	(hierarchical_label "SpareSW1"
+	(hierarchical_label "GimbalPanSW"
 		(shape input)
 		(at 168.91 88.9 0)

Commit message: Add reverse voltage protection circuit
Changed lines of the file:
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@@
 		(pin "24"
 		)
-		(pin "D"
+		(pin "D-"
 		)
 		(pin "39"

Commit message: Caught mislabeled pinout for AF after the recent pin change
Connections:
- net AFLED340 renamed AFLED365
Changed lines of the file:
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@@
 		)
 	)
-	(hierarchical_label "AFLED340"
+	(hierarchical_label "AFLED365"
 		(shape output)
 		(at 120.65 76.2 180)
