File: board/AugerBoard.kicad_pcb (KiCad board)
At the start: 2 copper layers, 96.5 x 88.9 mm, 88 parts, among them J1 RJ45_LED_Shielded, J2 Conn_01x04_MountingPin, J3 2002411212, J4 2002411212, J5 2002411212, J6 2002411212, J7 2002411212, Q1 BSS138, Q2 BSS138, Q3 BSS138, Q4 BSS138, Q5 BSS138, Q6 BSS138, Q7 BSS138, Q8 BSS138, Q9 BSS138, SW1 SW_Push, SW10 SW_SPDT, SW2 SW_Push, SW3 SW_Push, SW4 SW_Push, SW5 SW_Push, SW6 SW_Push, SW7 SW_Push, SW8 SW_Push, SW9 SW_Push, U1 OKI 5V, U2 Teensy4.1_DEV-16771, U3 ATA6561, U4 OKI 3V3, U5 ATA6561, U6 MAX3485

Commit message: Redesigning Layout
Parts:
- removed Conn16: Molex_uF_D_04, MRDT_Connectors:MOLEX_SL_04_Vertical
- removed the G*** at (147.3, 148.1)
- removed H5, H6: MountingHole, MountingHole:MountingHole_2.7mm
- removed J2: Conn_01x04_MountingPin, Connector_PinHeader_2.54mm:PinHeader_1x04_P2.54mm_Vertical
- removed R5: 120, Resistor_SMD:R_0603_1608Metric_Pad0.98x0.95mm_HandSolder
- removed U6: MAX3485, Package_SO:SOIC-8_3.9x4.9mm_P1.27mm
- added Conn7: Molex_SL_04, MRDT_Connectors:MOLEX_SL_04_Vertical, F.Cu at (135.4, 54.5)
- moved Conn5 63.0 mm to (198.1, 117.1)
- moved D12 63.0 mm to (201.2, 122.7)
- moved Q9 63.0 mm to (197.1, 122.7)
- moved Conn1 63.0 mm to (173.5, 142.0)
- moved Conn2 63.0 mm to (174.8, 117.1)
- moved Conn3 63.0 mm to (186.4, 117.1)
- moved Conn4 63.0 mm to (186.4, 129.8)
- moved Conn6 63.0 mm to (174.8, 129.8)
- moved D10 63.0 mm to (177.8, 122.7)
- moved D11 63.0 mm to (189.5, 122.7)
- moved D8 63.0 mm to (177.8, 135.4)
- moved D9 63.0 mm to (189.5, 135.4)
- moved Q6 63.0 mm to (185.5, 135.4)
- moved Conn10 63.0 mm to (209.8, 117.1)
- moved Q5 63.0 mm to (173.7, 135.4)
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Connections:
- net /Power/SpareMotorLED renamed /Power/Spare12VLED
- net /Servos/AFSparePWM renamed /Servos/SparePWM1
- net /Servos/SoilCacheSparePWM renamed /Servos/SparePWM2
- net /Soil Sensors & NPK/Moisture renamed /Soil Sensors/Moisture
- net /Teensy/AFSpareSW renamed /Teensy/SpareSW1
- net /Teensy/SCacheSpareSW renamed /Teensy/SpareSW2
- J1 pad 2: /Communications/T- -> Net-(C3-Pad2)
- J1 pad 3: Net-(C3-Pad2) -> /Communications/T-
- Q4 pad 1: /Power/AFSpareLED -> /Power/SpareLED2
- Q9 pad 1: /Power/CacheSpareLED -> /Power/SpareLED1
- U2 pad 0: /Communications/RXD1 -> /Communications/RXD2
- U2 pad 1: /Communications/TXD1 -> /Communications/TXD2
- U2 pad 13: /Soil Sensors & NPK/RE -> unconnected-(U2-SCK-Pad13)
- U2 pad 14: /Soil Sensors & NPK/DE -> /AF interface/AFWhiteLED
- U2 pad 15: /Soil Sensors & NPK/DI -> unconnected-(U2-A1-Pad15)
- U2 pad 19: /Communications/STBY2 -> /Communications/STBY1
- U2 pad 20: /Communications/TXD2 -> /Power/VescLED
- U2 pad 21: /Communications/RXD2 -> /Power/GantryLED
- U2 pad 22: /Power/VescLED -> /Communications/TXD1
- U2 pad 23: /Power/GantryLED -> /Communications/RXD1
- U2 pad 26: /Power/CacheSpareLED -> /Power/SpareLED2
- U2 pad 3: /Communications/STBY1 -> /Communications/STBY2
- U2 pad 30: /Power/AFSpareLED -> /Power/SpareLED1
- U2 pad 31: /AF interface/AFWhiteLED -> unconnected-(U2-CTX3-Pad31)
- U2 pad 38: /Soil Sensors & NPK/Temp -> /Soil Sensors/Temp
- U2 pad 41: /Soil Sensors & NPK/RO -> unconnected-(U2-A17-Pad41)
- U3 pad 1: /Communications/TXD1 -> /Communications/TXD2
- U3 pad 4: /Communications/RXD1 -> /Communications/RXD2
- U3 pad 8: /Communications/STBY1 -> /Communications/STBY2
- U5 pad 1: /Communications/TXD2 -> /Communications/TXD1
- U5 pad 4: /Communications/RXD2 -> /Communications/RXD1
- U5 pad 8: /Communications/STBY2 -> /Communications/STBY1
Routing:
- net +5V: track 278.0 -> 0.00 mm, vias 29 -> 0
- net +3.3V: track 192.9 -> 0.00 mm, vias 15 -> 0
- net Net-(U5-CANL): track 85.3 -> 0.00 mm, vias 2 -> 0
- net Net-(U5-CANH): track 84.9 -> 0.00 mm, vias 2 -> 0
- net Net-(U3-CANH): track 81.7 -> 0.00 mm, vias 4 -> 0
- net Net-(U3-CANL): track 81.6 -> 0.00 mm, vias 4 -> 0
- net /AF interface/AFWhiteLED: track 77.4 -> 0.00 mm, vias 1 -> 0
- net Net-(U6-A): track 75.3 -> 0.00 mm, vias 2 -> 0
- net Net-(U6-B): track 75.2 -> 0.00 mm, vias 2 -> 0
- net /Communications/LED: track 60.2 -> 0.00 mm, vias 1 -> 0
- net /Teensy/SoilDoorSW: track 57.6 -> 0.00 mm, vias 1 -> 0
- net /Teensy/AFLensSW: track 54.5 -> 0.00 mm, vias 1 -> 0
- net /Teensy/SpareSW1: track 52.8 -> 0.00 mm, vias 1 -> 0
- net /Teensy/GimbalTiltSW: track 52.5 -> 0.00 mm, vias 3 -> 0
- net /Teensy/GimbalPanSW: track 49.5 -> 0.00 mm, vias 1 -> 0
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Other:
- board text added: "12V"
- board text added: "AF Board"
- board text added: "SMoCo Board"
- board text added: "Spare 1"
- board text added: "Spare 2"
- board text added: "VESC Board"
- board text removed: "+12V"
- board text removed: "+3V3"
- board text removed: "+5V"
- board text removed: "AF Board Power"
- board text removed: "AF Spare"
- board text removed: "Auger VESC"
- board text removed: "Gantry Motor"
- board text removed: "NPK & pH"
- board text removed: "Soil Ch. Spare"
- board text removed: "Spare 12V Motor"
- board text removed: "Tmp"
- board text removed: "UA"
- board text removed: "UB"

Commit message: Temporary Designed Layout for review
Parts:
- moved Conn10 89.5 mm to (120.4, 120.9)
- moved R13 81.4 mm to (112.8, 136.1), turned to 0 degrees
- moved R14 80.4 mm to (124.5, 128.0), turned to 0 degrees
- moved Conn3 78.6 mm to (108.7, 129.0)
- moved Q8 77.7 mm to (108.7, 135.1)
- moved D11 77.6 mm to (112.8, 134.1)
- moved Q9 76.8 mm to (120.4, 127.0)
- moved D12 76.8 mm to (124.5, 126.0)
- moved Conn1 69.3 mm to (104.6, 149.9)
- moved R11 69.2 mm to (124.5, 144.8), turned to 0 degrees
- moved Conn4 66.5 mm to (120.4, 137.7)
- moved Q6 65.6 mm to (120.4, 143.8)
- moved D9 65.4 mm to (124.5, 142.7)
- moved D7 62.1 mm to (147.8, 126.0)
- moved R9 62.1 mm to (147.8, 128.0)
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Connections:
- U2 pad 10: /AF interface/AFLED490 -> /Teensy/GimbalPanSW
- U2 pad 11: /Power/AFFLED -> /Teensy/AFLensSW
- U2 pad 12: /Servos/AFLensPWM -> /Teensy/GantrySW
- U2 pad 13: unconnected-(U2-SCK-Pad13) -> /Servos/SciGimbalPan
- U2 pad 14: /AF interface/AFWhiteLED -> /Servos/SparePWM1
- U2 pad 15: unconnected-(U2-A1-Pad15) -> /Servos/SoilTrapdoorPWM
- U2 pad 16: /Teensy/SpareSW2 -> /Power/SpareLED1
- U2 pad 17: /Teensy/SoilDoorSW -> /Power/SoilTDLED
- U2 pad 18: /Teensy/GantrySW -> /Servos/SparePWM2
- U2 pad 19: /Communications/STBY1 -> /Servos/SciGimbalTilt
- U2 pad 2: /Power/Spare12VLED -> unconnected-(U2-OUT2-Pad2)
- U2 pad 20: /Power/VescLED -> /Power/GimbalTiltLED
- U2 pad 21: /Power/GantryLED -> /Power/SpareLED2
- U2 pad 24: /Servos/SciGimbalPan -> /Soil Sensors/Moisture
- U2 pad 25: /Power/GimbalPanLED -> /Soil Sensors/Temp
- U2 pad 26: /Power/SpareLED2 -> /Teensy/SpareSW_12V
- U2 pad 27: /Soil Sensors/Moisture -> /Communications/STBY1
- U2 pad 28: /Servos/SparePWM2 -> /Communications/STBY2
- U2 pad 29: /Servos/SparePWM1 -> /Teensy/Dir_Switch
- U2 pad 3: /Communications/STBY2 -> unconnected-(U2-LRCLK2-Pad3)
- U2 pad 30: /Power/SpareLED1 -> /Power/GantryLED
- U2 pad 33: /Teensy/Dir_Switch -> /Power/Spare12VLED
- U2 pad 34: /Teensy/GimbalTiltSW -> /Power/VescLED
- U2 pad 35: /Teensy/SpareSW1 -> /Power/AFFLED
- U2 pad 36: /Teensy/SpareSW_12V -> /Power/GimbalPanLED
- U2 pad 37: /Teensy/GimbalPanSW -> /Servos/AFLensPWM
- U2 pad 38: /Soil Sensors/Temp -> /AF interface/AFWhiteLED
- U2 pad 39: /Teensy/AFLensSW -> /AF interface/AFLED365
- U2 pad 4: /Power/SoilTDLED -> unconnected-(U2-BCLK2-Pad4)
- U2 pad 40: /Teensy/AugerSW -> /AF interface/AFLED405
- U2 pad 41: unconnected-(U2-A17-Pad41) -> /AF interface/AFLED490
- U2 pad 5: /Servos/SoilTrapdoorPWM -> /Teensy/SpareSW2
- U2 pad 6: /Servos/SciGimbalTilt -> /Teensy/GimbalTiltSW
- U2 pad 7: /Power/GimbalTiltLED -> /Teensy/SoilDoorSW
- U2 pad 8: /AF interface/AFLED365 -> /Teensy/AugerSW
- U2 pad 9: /AF interface/AFLED405 -> /Teensy/SpareSW1
Other:
- board size 96.5 x 88.9 mm -> 88.9 x 88.9 mm
- board text added: "Auger Board, Rev2 Mars Rover Design Team Missouri S&T, 2026 Blaydn Buckwalter"
- board text added: "Temperature"
- board text removed: "Auger Board, Rev1 Mars Rover Design Team Missouri S&T, 2026 Blaydn Buckwalter, Malachi Dascent"

Commit message: Temporary 2nd Auger Board
Parts:
- added C1: 10uF, Capacitor_SMD:C_0603_1608Metric_Pad1.08x0.95mm_HandSolder, F.Cu at (-76.6, 82.8)
- added C2: 10uF, Capacitor_SMD:C_0603_1608Metric_Pad1.08x0.95mm_HandSolder, F.Cu at (-81.7, 82.8)
- added C3: 0.1uF, Capacitor_SMD:C_0603_1608Metric_Pad1.08x0.95mm_HandSolder, F.Cu at (-91.7, 140.0)
- added C4: 10uF, Capacitor_SMD:C_0603_1608Metric_Pad1.08x0.95mm_HandSolder, F.Cu at (-65.9, 82.8)
- added C5: 10uF, Capacitor_SMD:C_0603_1608Metric_Pad1.08x0.95mm_HandSolder, F.Cu at (-71.0, 82.8)
- added Conn1: Molex_SL_05, MRDT_Connectors:MOLEX_SL_05_Vertical, F.Cu at (-74.5, 148.2)
- added Conn10: Molex_SL_03, MRDT_Connectors:MOLEX_SL_03_Vertical, F.Cu at (-58.8, 119.3)
- added Conn12: Molex_SL_02, MRDT_Connectors:MOLEX_SL_02_Vertical, F.Cu at (-90.8, 148.2)
- added Conn13: Molex_SL_02, MRDT_Connectors:MOLEX_SL_02_Vertical, F.Cu at (-82.7, 148.2)
- added Conn2: Molex_SL_03, MRDT_Connectors:MOLEX_SL_03_Vertical, F.Cu at (-47.1, 127.4)
- added Conn3: Molex_SL_03, MRDT_Connectors:MOLEX_SL_03_Vertical, F.Cu at (-70.5, 127.4)
- added Conn4: Molex_SL_03, MRDT_Connectors:MOLEX_SL_03_Vertical, F.Cu at (-58.8, 136.0)
- added Conn5: Molex_SL_03, MRDT_Connectors:MOLEX_SL_03_Vertical, F.Cu at (-35.4, 119.3)
- added Conn6: Molex_SL_03, MRDT_Connectors:MOLEX_SL_03_Vertical, F.Cu at (-35.9, 136.0)
- added Conn7: Molex_SL_04, MRDT_Connectors:MOLEX_SL_04_Vertical, F.Cu at (-39.0, 80.6)
- added Conn9: Molex_SL_03, MRDT_Connectors:MOLEX_SL_03_Vertical, F.Cu at (-36.4, 90.3)
- added D1: GREEN, LED_SMD:LED_0603_1608Metric_Pad1.05x0.95mm_HandSolder, F.Cu at (-92.3, 77.9)
- added D10: ORANGE, LED_SMD:LED_0603_1608Metric_Pad1.05x0.95mm_HandSolder, F.Cu at (-43.1, 132.5)
- added D11: ORANGE, LED_SMD:LED_0603_1608Metric_Pad1.05x0.95mm_HandSolder, F.Cu at (-66.4, 132.5)
- added D12: ORANGE, LED_SMD:LED_0603_1608Metric_Pad1.05x0.95mm_HandSolder, F.Cu at (-54.7, 124.3)
- added D13: MMSZ5240BT1G, MRDT_Devices:SOD-123_ONS-L, F.Cu at (-104.1, 70.0)
- added D2: GREEN, LED_SMD:LED_0603_1608Metric_Pad1.05x0.95mm_HandSolder, F.Cu at (-89.3, 77.9)
- added D3: GREEN, LED_SMD:LED_0603_1608Metric_Pad1.05x0.95mm_HandSolder, F.Cu at (-86.2, 77.9)
- added D4: ORANGE, LED_SMD:LED_0603_1608Metric_Pad1.05x0.95mm_HandSolder, F.Cu at (-93.3, 87.5)
- added D5: ORANGE, LED_SMD:LED_0603_1608Metric_Pad1.05x0.95mm_HandSolder, F.Cu at (-93.3, 98.4)
- added D6: ORANGE, LED_SMD:LED_0603_1608Metric_Pad1.05x0.95mm_HandSolder, F.Cu at (-93.3, 119.8)
- added D7: ORANGE, LED_SMD:LED_0603_1608Metric_Pad1.05x0.95mm_HandSolder, F.Cu at (-31.4, 124.3)
- added D8: ORANGE, LED_SMD:LED_0603_1608Metric_Pad1.05x0.95mm_HandSolder, F.Cu at (-31.9, 141.1)
- added D9: ORANGE, LED_SMD:LED_0603_1608Metric_Pad1.05x0.95mm_HandSolder, F.Cu at (-54.7, 141.1)
- added G***: LOGO, LOGO, F.Cu at (-47.1, 151.6)
- added H1: MountingHole, MRDT_Drill_Holes:4_40_Hole_Corner, F.Cu at (-35.9, 144.2)
- added H2: MountingHole, MRDT_Drill_Holes:4_40_Hole_Corner, F.Cu at (-106.6, 144.2)
- added H3: MountingHole, MRDT_Drill_Holes:4_40_Hole_Corner, F.Cu at (-106.6, 73.5)
- added H4: MountingHole, MRDT_Drill_Holes:4_40_Hole_Corner, F.Cu at (-35.9, 73.5)
- added J1: RJ45_LED_Shielded, MRDT_Connectors:RJ45_Teensy, F.Cu at (-117.6, 135.6)
- added J3: 2002411212, footprints:CONN_SD-76825-0100_02_MOL, F.Cu at (-103.5, 111.1)
- added J4: 2002411212, footprints:CONN_SD-76825-0100_02_MOL, F.Cu at (-103.5, 89.8)
- added J5: 2002411212, footprints:CONN_SD-76825-0100_02_MOL, F.Cu at (-103.5, 100.5)
- added J6: 2002411212, footprints:CONN_SD-76825-0100_02_MOL, F.Cu at (-103.5, 121.8)
- added J7: 2002411212, footprints:CONN_SD-76825-0100_02_MOL, F.Cu at (-103.5, 79.1)
- added MOSFET1: TPC8132_LQS, MRDT_Devices:SOP-8_TOS-L, F.Cu at (-99.4, 71.0)
- added Q1: BSS138, Package_TO_SOT_SMD:SOT-23, F.Cu at (-92.3, 91.6)
- added Q2: BSS138, Package_TO_SOT_SMD:SOT-23, F.Cu at (-92.3, 102.5)
- added Q3: BSS138, Package_TO_SOT_SMD:SOT-23, F.Cu at (-92.3, 123.8)
- added Q4: BSS138, Package_TO_SOT_SMD:SOT-23, F.Cu at (-35.4, 125.3)
- added Q5: BSS138, Package_TO_SOT_SMD:SOT-23, F.Cu at (-35.9, 142.1)
- added Q6: BSS138, Package_TO_SOT_SMD:SOT-23, F.Cu at (-58.8, 142.1)
- added Q7: BSS138, Package_TO_SOT_SMD:SOT-23, F.Cu at (-47.1, 133.5)
- added Q8: BSS138, Package_TO_SOT_SMD:SOT-23, F.Cu at (-70.5, 133.5)
- added Q9: BSS138, Package_TO_SOT_SMD:SOT-23, F.Cu at (-58.8, 125.3)
- added R1: 2.2k, Resistor_SMD:R_0603_1608Metric_Pad0.98x0.95mm_HandSolder, F.Cu at (-92.3, 81.7)
- added R10: 1.5k, Resistor_SMD:R_0603_1608Metric_Pad0.98x0.95mm_HandSolder, F.Cu at (-31.9, 143.1)
- added R11: 1.5k, Resistor_SMD:R_0603_1608Metric_Pad0.98x0.95mm_HandSolder, F.Cu at (-54.7, 143.1)
- added R12: 1.5k, Resistor_SMD:R_0603_1608Metric_Pad0.98x0.95mm_HandSolder, F.Cu at (-43.1, 134.5)
- added R13: 1.5k, Resistor_SMD:R_0603_1608Metric_Pad0.98x0.95mm_HandSolder, F.Cu at (-66.4, 134.5)
- added R14: 1.5k, Resistor_SMD:R_0603_1608Metric_Pad0.98x0.95mm_HandSolder, F.Cu at (-54.7, 126.4)
- added R15: 120, Resistor_SMD:R_0603_1608Metric_Pad0.98x0.95mm_HandSolder, F.Cu at (-77.7, 127.1)
- added R16: 120, Resistor_SMD:R_0603_1608Metric_Pad0.98x0.95mm_HandSolder, F.Cu at (-84.7, 127.1)
- added R2: 820, Resistor_SMD:R_0603_1608Metric_Pad0.98x0.95mm_HandSolder, F.Cu at (-89.3, 81.7)
- added R3: 330, Resistor_SMD:R_0603_1608Metric_Pad0.98x0.95mm_HandSolder, F.Cu at (-86.2, 81.7)
- added R4: 1k, Resistor_SMD:R_0603_1608Metric_Pad0.98x0.95mm_HandSolder, F.Cu at (-105.2, 73.4)
- added R6: 1.5k, Resistor_SMD:R_0603_1608Metric_Pad0.98x0.95mm_HandSolder, F.Cu at (-91.3, 87.5)
- added R7: 1.5k, Resistor_SMD:R_0603_1608Metric_Pad0.98x0.95mm_HandSolder, F.Cu at (-91.3, 98.4)
- added R8: 1.5k, Resistor_SMD:R_0603_1608Metric_Pad0.98x0.95mm_HandSolder, F.Cu at (-91.3, 119.8)
- added R9: 1.5k, Resistor_SMD:R_0603_1608Metric_Pad0.98x0.95mm_HandSolder, F.Cu at (-31.4, 126.4)
- added S1: SLW-913535-2A-SMT, MRDT_Switches:SW_SLW-913535-2A-SMT, F.Cu at (-81.2, 135.5)
- added SW1: SW_Push, Button_Switch_SMD:SW_SPST_TL3305A, F.Cu at (-57.8, 70.0)
- added SW10: SW_SPDT, Button_Switch_THT:SW_Slide_SPDT_Straight_CK_OS102011MS2Q, F.Cu at (-80.7, 89.8)
- added SW2: SW_Push, Button_Switch_SMD:SW_SPST_TL3305A, F.Cu at (-47.1, 70.0)
- added SW3: SW_Push, Button_Switch_SMD:SW_SPST_TL3305A, F.Cu at (-69.0, 89.8)
- added SW4: SW_Push, Button_Switch_SMD:SW_SPST_TL3305A, F.Cu at (-47.1, 76.6)
- added SW5: SW_Push, Button_Switch_SMD:SW_SPST_TL3305A, F.Cu at (-57.8, 76.6)
- added SW6: SW_Push, Button_Switch_SMD:SW_SPST_TL3305A, F.Cu at (-57.8, 89.8)
- added SW7: SW_Push, Button_Switch_SMD:SW_SPST_TL3305A, F.Cu at (-47.1, 89.8)
- added SW8: SW_Push, Button_Switch_SMD:SW_SPST_TL3305A, F.Cu at (-57.8, 83.2)
- added SW9: SW_Push, Button_Switch_SMD:SW_SPST_TL3305A, F.Cu at (-47.1, 83.2)
- added U1: OKI 5V, MRDT_Devices:OKI_Horizontal, F.Cu at (-76.6, 80.1)
- added U2: Teensy4.1_DEV-16771, MRDT_Shields:Teensy_4_1_Ethernet, F.Cu at (-57.8, 104.5)
- added U3: ATA6561, Package_SO:SOIC-8_3.9x4.9mm_P1.27mm, F.Cu at (-84.7, 122.3)
- added U4: OKI 3V3, MRDT_Devices:OKI_Horizontal, F.Cu at (-65.9, 80.1)
- added U5: ATA6561, Package_SO:SOIC-8_3.9x4.9mm_P1.27mm, F.Cu at (-77.6, 122.3)
- moved G*** 99.8 mm to (211.6, 112.0)
- moved Conn3 32.3 mm to (129.0, 103.9)
- moved D11 32.3 mm to (133.1, 109.0)
- moved R13 32.3 mm to (133.1, 111.0)
- moved Q8 32.3 mm to (129.0, 110.0)
- moved U5 32.1 mm to (99.6, 156.0), turned to 180 degrees
- moved SW2 32.0 mm to (101.6, 81.3)
- moved U2 31.3 mm to (99.6, 128.5), turned to 90 degrees
- moved Conn2 30.8 mm to (114.3, 103.9)
- moved D10 30.8 mm to (118.4, 109.0)
- moved R12 30.8 mm to (118.4, 111.0)
- moved Q7 30.8 mm to (114.3, 110.0)
- moved R15 27.9 mm to (94.7, 155.8), turned to -90 degrees
- moved U3 25.4 mm to (99.6, 148.8), turned to 180 degrees
- moved Conn6 24.4 mm to (129.0, 117.9)
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Other:
- board size 88.9 x 88.9 mm -> 257.9 x 95.6 mm

Commit message: minor trace routing started
Parts:
- moved Conn13 9.76 mm to (83.3, 157.0)
- moved R15 6.86 mm to (94.7, 149.0)
- moved U5 6.86 mm to (99.6, 149.1)
- moved R16 6.60 mm to (94.7, 155.4)
- moved U3 6.60 mm to (99.6, 155.4)
- moved S1 5.08 mm to (81.3, 147.3), turned to 0 degrees
- moved C3 4.37 mm to (85.0, 138.0)
- moved J1 4.37 mm to (59.1, 133.7)
- moved J6 4.06 mm to (75.7, 119.4)
- moved D6 3.66 mm to (85.9, 117.8)
- moved R8 3.66 mm to (87.9, 117.8), turned to 90 degrees
- moved Q3 3.66 mm to (86.9, 121.8)
- moved J3 3.05 mm to (75.7, 109.7)
- moved C4 2.50 mm to (123.7, 69.6), turned to 0 degrees
- moved C5 2.50 mm to (123.7, 74.7), turned to 0 degrees
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Routing:
- net +5V: track 0.00 -> 112.6 mm, vias 0 -> 5
- net +12V: track 0.00 -> 50.2 mm, vias 0 -> 5
- net Net-(MOSFET1-D): track 0.00 -> 10.5 mm
- net Net-(MOSFET1-G): track 0.59 -> 4.66 mm
- net +3.3V: track 0.00 -> 2.44 mm
- net Net-(D3-A): track 0.00 -> 2.02 mm
- net Net-(D2-A): track 0.00 -> 2.02 mm
- net Net-(D1-A): track 0.00 -> 2.02 mm
