File: board/communications.kicad_sch (KiCad schematic)
At the start: 9 parts, among them J1 RJ45_LED_Shielded, U3 ATA6561, U5 ATA6561

Commit message: Redesigning Layout
Connections:
- net RXD1: now also U5.4 (RXD); no longer U3.4 (RXD)
- net RXD2: now also U3.4 (RXD); no longer U5.4 (RXD)
- net STBY1: now also U5.8 (STBY); no longer U3.8 (STBY)
- net STBY2: now also U3.8 (STBY); no longer U5.8 (STBY)
- net T-: now also J1.3; no longer J1.2
- net TXD1: now also U5.1 (TXD); no longer U3.1 (TXD)
- net TXD2: now also U3.1 (TXD); no longer U5.1 (TXD)
- net at C3.2, J1.5: now also J1.2; no longer J1.3
Changed lines of the file:
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@@
-	)
-	(junction
-		(at 44.45 63.5)
-		(diameter 0)
-		(color 0 0 0 0)
 	)
 	(junction
@@
 	)
 	(junction
+		(at 41.91 63.5)
+		(diameter 0)
+		(color 0 0 0 0)
+	)
+	(junction
 		(at 130.81 58.42)
 		(diameter 0)
@@
 	(wire
 		(pts
-			(xy 44.45 50.8) (xy 44.45 63.5)
-		)
-		(stroke
-			(width 0)
-			(type default)
-		)
-	)
-	(wire
-		(pts
 			(xy 127 95.25) (xy 127 97.79)
 		)
@@
 	(wire
 		(pts
+			(xy 44.45 50.8) (xy 44.45 52.07)
+		)
+		(stroke
+			(width 0)
+			(type default)
+		)
+	)
+	(wire
+		(pts
+			(xy 41.91 63.5) (xy 49.53 63.5)
+		)
+		(stroke
+			(width 0)
+			(type default)
+		)
+	)
+	(wire
+		(pts
 			(xy 127 72.39) (xy 137.16 72.39)
 		)
@@
 	(wire
 		(pts
+			(xy 41.91 50.8) (xy 41.91 63.5)
+		)
+		(stroke
+			(width 0)
+			(type default)
+		)
+	)
+	(wire
+		(pts
 			(xy 111.76 33.02) (xy 111.76 39.37)
 		)
@@
 	(wire
 		(pts
-			(xy 38.1 63.5) (xy 44.45 63.5)
+			(xy 38.1 63.5) (xy 41.91 63.5)
 		)
 		(stroke
@@
 	(wire
 		(pts
-			(xy 41.91 50.8) (xy 41.91 52.07)
-		)
-		(stroke
-			(width 0)
-			(type default)
-		)
-	)
-	(wire
-		(pts
 			(xy 27.94 40.64) (xy 27.94 63.5)
 		)
@@
 	(wire
 		(pts
-			(xy 49.53 63.5) (xy 44.45 63.5)
-		)
-		(stroke
-			(width 0)
-			(type default)
-		)
-	)
-	(wire
-		(pts
 			(xy 34.29 40.64) (xy 27.94 40.64)
 		)
@@
 		)
 	)
-	(hierarchical_label "STBY2"
+	(hierarchical_label "STBY1"
 		(shape input)
 		(at 100.33 97.79 180)
@@
 	(hierarchical_label "T-"
 		(shape input)
-		(at 41.91 52.07 270)
-		(effects
-			(font
-				(size 1.27 1.27)
-			)
-			(justify right)
-		)
-	)
-	(hierarchical_label "TXD2"
+		(at 44.45 52.07 270)
+		(effects
+			(font
+				(size 1.27 1.27)
+			)
+			(justify right)
+		)
+	)
+	(hierarchical_label "TXD1"
 		(shape input)
 		(at 100.33 102.87 180)
+		(effects
+			(font
+				(size 1.27 1.27)
+			)
+			(justify right)
+		)
+	)
+	(hierarchical_label "RXD1"
+		(shape output)
+		(at 100.33 105.41 180)
 		(effects
 			(font
@@
 	(hierarchical_label "RXD2"
 		(shape output)
-		(at 100.33 105.41 180)
-		(effects
-			(font
-				(size 1.27 1.27)
-			)
-			(justify right)
-		)
-	)
-	(hierarchical_label "RXD1"
-		(shape output)
 		(at 100.33 55.88 180)
 		(effects
@@
 		)
 	)
-	(hierarchical_label "TXD1"
+	(hierarchical_label "TXD2"
 		(shape input)
 		(at 100.33 53.34 180)
@@
 		)
 	)
-	(hierarchical_label "STBY1"
+	(hierarchical_label "STBY2"
 		(shape input)
 		(at 100.33 48.26 180)
